Commit message: test updated

File: SNS Training/combined.urdf (robot description, URDF)
Before this commit: robot GantryAssembly_NoGrasper, 14 links, 13 joints
Links:
- link BasePlate: geometry collision mesh filename=c:\Users\Yanjun\Documents\Aplysia_soft_grasper_deformable_o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 scale=1.00000 1.00000 1.00000; visual mesh filename=c:\Users\Yanjun\Documents\Aplysia_soft_grasper_deformable_o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 scale=1.00000 1.00000 1.00000
- link GrasperBase: geometry collision mesh filename=c:\Users\Yanjun\Documents\Aplysia_soft_grasper_deformable_o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 scale=1.00000 1.00000 1.00000; visual mesh filename=c:\Users\Yanjun\Documents\Aplysia_soft_grasper_deformable_o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 scale=1.00000 1.00000 1.00000
- link LeftUpright: geometry collision mesh filename=c:\Users\Yanjun\Documents\Aplysia_soft_grasper_deformable_o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 scale=1.00000 1.00000 1.00000; visual mesh filename=c:\Users\Yanjun\Documents\Aplysia_soft_grasper_deformable_o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 scale=1.00000 1.00000 1.00000
- link RightUpright: geometry collision mesh filename=c:\Users\Yanjun\Documents\Aplysia_soft_grasper_deformable_o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 scale=1.00000 1.00000 1.00000; visual mesh filename=c:\Users\Yanjun\Documents\Aplysia_soft_grasper_deformable_o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 scale=1.00000 1.00000 1.00000
- link ZBar: geometry collision mesh filename=c:\Users\Yanjun\Documents\Aplysia_soft_grasper_deformable_o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 scale=1.00000 1.00000 1.00000; visual mesh filename=c:\Users\Yanjun\Documents\Aplysia_soft_grasper_deformable_o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 scale=1.00000 1.00000 1.00000
- link base_link_gantry: geometry collision mesh filename=c:\Users\Yanjun\Documents\Aplysia_soft_grasper_deformable_o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 scale=1.00000 1.00000 1.00000; visual mesh filename=c:\Users\Yanjun\Documents\Aplysia_soft_grasper_deformable_o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 scale=1.00000 1.00000 1.00000
